Commit message: adding SLAM mapping using RTAB package to the my_robot

File: urdf/my_robot.xacro (robot description, xacro)
@@ -159,5 +159,5 @@
   <link name='hokuyo'>
     <pose>0 0 0 0 0 0</pose>
-	<origin xyz="0.0 0.0 0.0" rpy=" 0 0 0"/>
+    <origin xyz="0.0 0.0 0.0" rpy=" 0 0 0"/>
     <inertial>
       <mass value="1e-5"/>
@@ -182,3 +182,10 @@
     </visual>
   </link>
+  <joint name="camera_optical_joint" type="fixed">
+    <origin xyz="0 0 0" rpy="-1.5707 0 -1.5707"/>
+    <parent link="camera"/>
+    <child link="camera_link_optical"/>
+  </joint>
+  <link name="camera_link_optical">
+  </link>
 </robot>
